Commit message: Did the TCP adjustment to tool0 so the flange is now just further away. But this is only in moveit

File: packages/ur16e_moveit_config/config/ur16e.urdf.xacro (robot description, xacro)
@@ -277,5 +277,5 @@
   <joint name="flange-tool0" type="fixed">
     <!-- default toolframe - X+ left, Y+ up, Z+ front -->
-    <origin rpy="1.5707963267948966 0 1.5707963267948966" xyz="0 0 0"/>
+    <origin rpy="1.5707963267948966 0 1.5707963267948966" xyz="0 0 0.563"/>
     <parent link="flange"/>
     <child link="tool0"/>

Commit message: fix(calibration): lower minimum detection confidence to improve detection reliability fix(vision): update model path comment for clarity fix(urdf): adjust tool0 joint position for better flange alignment

File: packages/ur16e_moveit_config/config/ur16e.urdf.xacro (robot description, xacro)
@@ -277,5 +277,5 @@
   <joint name="flange-tool0" type="fixed">
     <!-- default toolframe - X+ left, Y+ up, Z+ front -->
-    <origin rpy="1.5707963267948966 0 1.5707963267948966" xyz="0 0 0.563"/>
+    <origin rpy="1.5707963267948966 0 1.5707963267948966" xyz="0.150 0 0"/>
     <parent link="flange"/>
     <child link="tool0"/>
