Commit message: feat(moveit): model the E-Pick gripper for collision on both arms
Without it MoveIt believes the flange is bare and plans the wrist to fold the
gripper back into the arm, the table or the camera. Adds an "epick" link fixed
to the flange in both URDFs: two measured cylinders (body 115 mm, D85; cup
D30), stopping 10 mm short of tool0 so the cup lip can still touch objects and
the final pick descent is not rejected as a collision.

Each SRDF disables epick only against wrist_3_link, which it is bolted to.
Random sampling over 5000 states hit the upper arm and forearm ~11% each, so
every other pair stays enabled.

The grasped-object box attached at tool0 now lists epick as a touch link:
the held object sits against the cup, so that contact is expected, and without
it every post-grasp move started in collision.

test_robot_profiles.py asserts the link, its flange mount, the short-of-tool0
extent and the single SRDF exemption on every arm, since a URDF regeneration
drops the hand edit silently.

Co-Authored-By: Claude Opus 5 <noreply@anthropic.com>

File: packages/recycle_bot_moveit_config/config/ur16e/ur16e.urdf.xacro (robot description, xacro)
@@ -281,3 +281,45 @@
     <child link="tool0"/>
   </joint>
+  <!-- Robotiq E-Pick collision geometry. NOT stock ur_description, and dropped
+       by a regeneration like the tool0 offset above. Identical to, and fully
+       documented in, ur3e/ur3e.urdf.xacro — keep the two in step.
+       Measured 2026-09-11: body 115 mm long, 85 mm diameter; suction cup
+       40 mm long, 30 mm diameter. -->
+  <link name="epick">
+    <visual>
+      <origin rpy="0 1.5707963267948966 0" xyz="0.0575 0 0"/>
+      <geometry>
+        <cylinder radius="0.0425" length="0.115"/>
+      </geometry>
+      <material name="epick_grey">
+        <color rgba="0.35 0.35 0.38 1.0"/>
+      </material>
+    </visual>
+    <visual>
+      <origin rpy="0 1.5707963267948966 0" xyz="0.1275 0 0"/>
+      <geometry>
+        <cylinder radius="0.015" length="0.025"/>
+      </geometry>
+      <material name="epick_grey">
+        <color rgba="0.35 0.35 0.38 1.0"/>
+      </material>
+    </visual>
+    <collision>
+      <origin rpy="0 1.5707963267948966 0" xyz="0.0575 0 0"/>
+      <geometry>
+        <cylinder radius="0.0425" length="0.115"/>
+      </geometry>
+    </collision>
+    <collision>
+      <origin rpy="0 1.5707963267948966 0" xyz="0.1275 0 0"/>
+      <geometry>
+        <cylinder radius="0.015" length="0.025"/>
+      </geometry>
+    </collision>
+  </link>
+  <joint name="flange-epick" type="fixed">
+    <parent link="flange"/>
+    <child link="epick"/>
+    <origin rpy="0 0 0" xyz="0 0 0"/>
+  </joint>
 </robot>

File: packages/recycle_bot_moveit_config/config/ur3e/ur3e.urdf.xacro (robot description, xacro)
@@ -292,3 +292,63 @@
     <child link="tool0"/>
   </joint>
+  <!-- Robotiq E-Pick collision geometry. NOT stock ur_description: the second
+       hand edit in this file, alongside the tool0 offset above, and dropped the
+       same way by a regeneration. Identical in ur16e/ur16e.urdf.xacro — the
+       gripper is the same on both arms.
+       Without it MoveIt believes the flange is bare, and happily plans the wrist
+       to fold the gripper back into the arm, the table or the camera.
+       Frame: the flange's own, whose X axis points out of the tool face — tool0
+       is at x = 0.150. URDF cylinders run along their local Z, so rpy pitches
+       them +90 deg onto X.
+       Two cylinders, flange face outward:
+         body        x 0.000 .. 0.115   radius 0.0425
+         suction cup x 0.115 .. 0.140   radius 0.015
+       MEASURED 2026-09-11: body 115 mm long from the flange face, 85 mm
+       diameter; suction cup 40 mm long, 30 mm diameter.
+       115 + 40 = 155 mm, 5 mm past tool0 at 150. The 150 was verified with the
+       cup resting on the table (see test_tool_offset_verified_against_a_physical
+       _surface), so it stays: the cup compresses on contact and/or its fitting
+       overlaps the body. Either way the cup occupies roughly 0.115 .. 0.150.
+       The model stops 10 mm short of tool0 on purpose. The cup lip is what
+       touches the object, and the table under a flat one, so modelling it would
+       make every pick's final LIN descent "collide" and be rejected. The
+       grasped-object box rec_bot_control attaches at tool0 lists epick as a touch
+       link for the same reason. Keep the cup end short of 0.150. -->
+  <link name="epick">
+    <visual>
+      <origin rpy="0 1.5707963267948966 0" xyz="0.0575 0 0"/>
+      <geometry>
+        <cylinder radius="0.0425" length="0.115"/>
+      </geometry>
+      <material name="epick_grey">
+        <color rgba="0.35 0.35 0.38 1.0"/>
+      </material>
+    </visual>
+    <visual>
+      <origin rpy="0 1.5707963267948966 0" xyz="0.1275 0 0"/>
+      <geometry>
+        <cylinder radius="0.015" length="0.025"/>
+      </geometry>
+      <material name="epick_grey">
+        <color rgba="0.35 0.35 0.38 1.0"/>
+      </material>
+    </visual>
+    <collision>
+      <origin rpy="0 1.5707963267948966 0" xyz="0.0575 0 0"/>
+      <geometry>
+        <cylinder radius="0.0425" length="0.115"/>
+      </geometry>
+    </collision>
+    <collision>
+      <origin rpy="0 1.5707963267948966 0" xyz="0.1275 0 0"/>
+      <geometry>
+        <cylinder radius="0.015" length="0.025"/>
+      </geometry>
+    </collision>
+  </link>
+  <joint name="flange-epick" type="fixed">
+    <parent link="flange"/>
+    <child link="epick"/>
+    <origin rpy="0 0 0" xyz="0 0 0"/>
+  </joint>
 </robot>
